Commit message: Stage 2, milestone 2.2

File: urdf/agric_orion.xacro (robot description, xacro)
@@ -82,3 +82,44 @@
       </plugin>
   </gazebo>
+      <joint name='lidar_joint' type='fixed'>
+        <parent link="base_link"/>
+        <child link="lidar_link"/>
+        <origin xyz="0.15 0 0.1" rpy="0 0 0"/>
+      </joint>
+      <link name="lidar_link">
+        <visual>
+          <geometry><cylinder radius="0.03" length="0.05"/></geometry>
+        </visual>
+        <collision>
+          <geometry><cylinder radius="0.03" length="0.05"/></geometry>
+        </collision>
+        <inertial>
+          <mass value="0.05"/>
+          <origin xyz="0 0 0"/>
+          <inertia ixx="0.00001" ixy="0" ixz="0" iyy="0.00001" iyz="0" izz="0.00001"/>
+        </inertial>
+      </link>
+      <gazebo reference="lidar_link">
+        <sensor name="lidar_sensor" type="gpu_lidar">
+          <pose>0 0 0 0 0 0</pose>
+          <topic>scan</topic>
+          <update_rate>10</update_rate>
+          <always_on>true</always_on>
+          <visualize>true</visualize>
+          <gz_frame_id>lidar_link</gz_frame_id>
+          <lidar>
+            <scan>
+              <horizontal>
+                <samples>360</samples>
+                <min_angle>-3.14159</min_angle>
+                <max_angle>3.14159</max_angle>
+              </horizontal>
+            </scan>
+            <range>
+              <min>0.12</min>
+              <max>10.0</max>
+            </range>
+          </lidar>
+        </sensor>
+      </gazebo>
 </robot>

Commit message: End of stage 2 , lesson learnt with readme file

File: urdf/agric_orion.xacro (robot description, xacro)
@@ -80,5 +80,9 @@
         name="gz::sim::systems::JointStatePublisher">
         <topic>joint_states</topic>
-      </plugin>
+    </plugin>
+    <plugin
+      filename="gz-sim-imu-system"
+      name="gz::sim::systems::Imu">
+    </plugin>
   </gazebo>
       <joint name='lidar_joint' type='fixed'>
@@ -123,3 +127,68 @@
         </sensor>
       </gazebo>
+  <joint name="imu_joint" type="fixed">
+    <parent link="base_link"/>
+    <child link ="imu_link"/>
+    <origin xyz="0 0 0.08" rpy="0 0 0"/>
+  </joint>
+  <link name="imu_link">
+    <visual>
+      <geometry><box size="0.02 0.02 0.02"/></geometry>
+    </visual>
+    <collision>
+      <geometry><box size="0.02 0.02 0.02"/></geometry>
+    </collision>
+    <inertial>
+      <mass value="0.01"/>
+      <origin xyz="0 0 0 "/>
+      <inertia ixx="0.000001" ixy="0" ixz="0" iyy="0.000001" iyz="0" izz="0.000001"/>
+    </inertial>
+  </link>
+    <gazebo reference ="imu_link">
+      <sensor name="imu" type="imu">
+        <topic>imu</topic>
+        <update_rate>10</update_rate>
+        <always_on>true</always_on>
+        <gz_frame_id>imu_link</gz_frame_id>
+      </sensor>
+    </gazebo>
+    <joint name="camera_joint" type="fixed">
+      <parent link="base_link"/>
+      <child link="camera_link"/>
+      <origin xyz= "0.2 0 0.05" rpy="0 0 0"/>
+    </joint>
+    <link name="camera_link">
+      <visual>
+        <geometry><cylinder radius="0.03" length="0.05"/></geometry>
+      </visual>
+      <collision>
+        <geometry><cylinder radius="0.03" length="0.05"/></geometry>
+      </collision>
+      <inertial>
+        <mass value="0.01" />
+        <origin xyz="0 0 0"/>
+        <inertia ixx="0.000001" ixy="0" ixz="0" iyy="0.000001" iyz="0" izz="0.000001"/>
+      </inertial>
+    </link>
+    <gazebo reference="camera_link">
+      <sensor name="camera" type="camera">
+        <topic>camera</topic>
+        <update_rate>10</update_rate>
+        <always_on>true</always_on>
+        <visualize>true</visualize>
+        <gz_frame_id>camera_link</gz_frame_id>
+        <camera>
+          <horizontal_fov>1.3</horizontal_fov>
+          <image>
+            <width>640</width>
+            <height>480</height>
+            <format>R8G8B8</format>
+          </image>
+          <clip>
+            <near>0.08</near>
+            <far>80</far>
+          </clip>
+        </camera>
+      </sensor>
+    </gazebo>
 </robot>
